File: 3V3To5VConversion.kicad_sch (KiCad schematic)
At the start: 15 parts, among them Q1 PMBT2222A,215, Q2 PMBT2222A,215, Q3 PMBT2222A,215, Q4 PMBT2222A,215, Q5 PMBT2222A,215, Q6 PMBT2222A,215, U1 74AHC04

Commit message: Add files via upload
Schematic and gerbers for a Gotek(?) compatible with an Artery AT32F435RGT7 chip and a 26 Pin FFC connector.
Used SFRKC30.AT4.35 PCB for most of the schematic and layout but used SFRC2D.B PCB for the 26 Pin FFC connections.
Used photographs and a multimeter along with removing U1 and U3 on the SFRKC30.AT4.35 to get to the traces underneath.
Where possible I followed the original PCB routing of the SFRKC30.AT4.35 but Kicad has some different rules for trace widths (between pins 5&6 of U8 which isn't fitted).
Removed L3 Green LED and changed R21 to 12K to reduce it's brightness. Also increased the pad sizes for the diode D1D to make it easier to hand solder. Minor changes to silk screen.
Other:
- title: Gotek(?) SMD Handrawn Schematic, Layout and Gerbers -> Gotek(?) Handrawn Schematic, Layout and Gerbers
Changed lines of the file:
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@@
 	(paper "A4")
 	(title_block
-		(title "Gotek(?) SMD Handrawn Schematic, Layout and Gerbers")
-		(date "2025-03-06")
-		(rev "1.0")
+		(title "Gotek(?) Handrawn Schematic, Layout and Gerbers")
+		(date "2025-04-11")
+		(rev "1.1")
 		(company "LiveBoxAndy")
 		(comment 1 "chip were removed to allow the routing underneath to be checked.")
 		(comment 2 "with the cable interface from an SFR1M44-DU26 (SFRC2D.B). The processor and the 74 ")
 		(comment 3 "Based on pictures and meter readings of an SRFKC30.AT4.35 for the processor bits mated")
-		(comment 4 "Changed to use all surface mount components.")
+		(comment 4 "Changed R21 to 12K to reduce brightness.")
 	)
 	(junction
