File: Gotek.kicad_sch (KiCad schematic)
At the start: 53 parts, among them J4 M20-8760542P, J5 M20-8760442, J7 OLED, J8 RotaryEncoder, P1 2005280260, P3 USB_A, U3 AT32F435RGT7, U4 AMS1117-3.3, U8 SST25VF016B-50-4C-S2AF, Y1 8Mhz

Commit message: Add files via upload
Schematic and gerbers for a Gotek(?) compatible with an Artery AT32F435RGT7 chip and a 26 Pin FFC connector.
Used SFRKC30.AT4.35 PCB for most of the schematic and layout but used SFRC2D.B PCB for the 26 Pin FFC connections.
Used photographs and a multimeter along with removing U1 and U3 on the SFRKC30.AT4.35 to get to the traces underneath.
Where possible I followed the original PCB routing of the SFRKC30.AT4.35 but Kicad has some different rules for trace widths (between pins 5&6 of U8 which isn't fitted).
Removed L3 Green LED and changed R21 to 12K to reduce it's brightness. Also increased the pad sizes for the diode D1D to make it easier to hand solder. Minor changes to silk screen.
Parts:
- removed J4: M20-8760542P, Gotek:HUSSP10W64P254_2X5_1270X500X1043P, symbol Gotek:M20-8760542P
- removed J5: M20-8760442, Gotek:M208760442, symbol Gotek:M20-8760442
- removed J8: RotaryEncoder, Gotek:610106249121, symbol Gotek:6101XX249121_610106249121
- added J10: Conn_01x04_Pin, Connector_PinHeader_2.54mm:PinHeader_1x04_P2.54mm_Vertical, symbol Connector:Conn_01x04_Pin
- added J3: Conn_01x03_Pin, Connector_PinHeader_2.54mm:PinHeader_1x03_P2.54mm_Vertical, symbol Connector:Conn_01x03_Pin
- added J4: Conn_01x02_Pin, Connector_PinHeader_2.54mm:PinHeader_1x02_P2.54mm_Vertical, symbol Connector:Conn_01x02_Pin
- added J5, JA1, JB1, JC1: Conn_01x02, Connector_PinHeader_2.54mm:PinHeader_1x02_P2.54mm_Vertical, symbol Connector:Conn_01x02_Pin
- added J8: RotaryEncoder, Connector_PinHeader_2.54mm:PinHeader_2x02_P2.54mm_Horizontal, symbol Connector:Conn_01x04_Pin
- added JD1, JE1: Conn_01x02_Pin, Connector_PinHeader_2.54mm:PinHeader_1x02_P2.54mm_Horizontal, symbol Connector:Conn_01x02_Pin
- added JK1, JKA1: Conn_01x02, Connector_PinHeader_2.54mm:PinHeader_2x01_P2.54mm_Horizontal, symbol Connector:Conn_01x02_Pin
- C1, C19: value 47uF -> 100uF; footprint Capacitor_Tantalum_SMD:CP_EIA-3528-21_Kemet-B_Pad1.50x2.35mm_HandSolder -> Capacitor_THT:CP_Radial_D5.0mm_P2.50mm
- C17: value 47uF -> 100uF; footprint Capacitor_Tantalum_SMD:CP_EIA-3528-21_Kemet-B_Pad1.50x2.35mm_HandSolder -> Capacitor_THT:CP_Radial_D5.0mm_P2.50mm; now not fitted
- J7: footprint Gotek:610106249121 -> Connector_PinHeader_2.54mm:PinHeader_2x02_P2.54mm_Horizontal; symbol Gotek:6101XX249121_610106249121 -> Connector:Conn_01x04_Pin
- L3: footprint Gotek:APT2012PGW -> LED_THT:LED_D4.0mm; symbol Gotek:APT2012PGW -> Device:LED; Height 0.85 -> (none); Manufacturer_Name Kingbright -> (none); Manufacturer_Part_Number APT2012PGW -> (none); Mouser Part Number 604-APT2012PGW -> (none); Mouser Price/Stock https://www.mouser.co.uk/ProductDetail/Kingbright/APT2012PG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 -> (none); now not fitted
- L4: footprint Gotek:APT2012PGW -> LED_THT:LED_D4.0mm; symbol Gotek:APT2012PGW -> Device:LED; Height 0.85 -> (none); Manufacturer_Name Kingbright -> (none); Manufacturer_Part_Number APT2012PGW -> (none); Mouser Part Number 604-APT2012PGW -> (none); Mouser Price/Stock https://www.mouser.co.uk/ProductDetail/Kingbright/APT2012PG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 -> (none)
- L5: footprint Gotek:HSMCC177 -> LED_THT:LED_D4.0mm; symbol Gotek:HSMC-C177 -> Device:LED; Height 0.5 -> (none); Manufacturer_Name Avago Technologies -> (none); Manufacturer_Part_Number HSMC-C177 -> (none); Mouser Part Number 630-HSMC-C177 -> (none); Mouser Price/Stock https://www.mouser.co.uk/ProductDetail/Broadcom-Avago/HSMC-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 -> (none)
- MO1: footprint Gotek:M208900705 -> Connector_PinHeader_2.54mm:PinHeader_1x03_P2.54mm_Horizontal; symbol Gotek:M20-8900705 -> Connector:Conn_01x03_Pin; Height 3.61 -> (none); Manufacturer_Name Harwin -> (none); Manufacturer_Part_Number M20-8900705 -> (none); Mouser Part Number 855-M20-8900705 -> (none); Mouser Price/Stock https://www.mouser.co.uk/ProductDetail/Harwin/M20-8900705?q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 -> (none)
- P3: footprint Gotek:USB1046GF0190LBA -> Connector_USB:USB_A_Molex_67643_Horizontal; symbol Gotek:USB1046-GF-0190-L-B-A -> Connector:USB_A; Height 7.2 -> (none); Manufacturer_Name GCT (GLOBAL CONNECTOR TECHNOLOGY) -> (none); Manufacturer_Part_Number USB1046-GF-0190-L-B-A -> (none); Mouser Part Number 640-USB1046GF0190LBA -> (none); Mouser Price/Stock https://www.mouser.co.uk/ProductDetail/GCT/USB1046-GF-0190-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 -> (none)
- R21: value 1K -> 12K
- S3, S4: value SKRTLAE010 -> SKHHANA010; footprint Gotek:SKRTLAE010 -> Gotek:SKHHLQA010; symbol Gotek:SKRTLAE010 -> Gotek:SKHHANA010; Height 3.3 -> (none); Manufacturer_Part_Number SKRTLAE010 -> SKHHANA010; Mouser Part Number 688-SKRTLA -> 688-SKHHAN; Mouser Price/Stock https://www.mouser.co.uk/ProductDetail/Alps-Alpine/SKRTLAE0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 -> https://www.mouser.co.uk/ProductDetail/Alps-Alpine/SKHHANA0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
- U8: now not fitted
- Y1: footprint Gotek:LFXTAL050985Bulk -> Crystal:Crystal_HC18-U_Vertical; symbol Gotek:LFXTAL050985Bulk -> Device:Crystal; Height 4.3 -> (none); Manufacturer_Name IQD -> (none); Manufacturer_Part_Number LFXTAL050985Bulk -> (none); Mouser Part Number 449-LFXTAL050985BULK -> (none); Mouser Price/Stock https://www.mouser.com/Search/Refine.aspx?Keyword=449-LFXTA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 -> (none)
Connections:
- net +3.3V: now also J7.4 (Pin_4), J3.2 (Pin_2); no longer J7.5
- net +5V: now also J10.2 (Pin_2), J8.4 (Pin_4)
- net DINST: now also P1.11, PU14.1, JD1.2 (Pin_2); no longer MO1.3
- net DRVSEL: now also MO1.1 (Pin_1); no longer MO1.7
- net ENC1: now also J8.1 (Pin_1)
- net ENC2: now also J8.2 (Pin_2)
- net ENCSW: now also JK1.1 (Pin_1)
- net GND: now also J7.3 (Pin_3), P3.5 (Shield), S3.4, S4.4, J10.1 (Pin_1), J5.2 (Pin_2), J8.3 (Pin_3), JA1.2 (Pin_2), JB1.2 (Pin_2), JC1.2 (Pin_2), JD1.1 (Pin_1), JE1.1 (Pin_1); no longer J7.6, MO1.2, MO1.4, P3.MH1, P3.MH2, S3.MP1, S3.MP2, S4.MP1, S4.MP2
- net HDOUT: now also JE1.2 (Pin_2); no longer MO1.1
- net I2C2_CLK: now also J7.1 (Pin_1), L3.1 (K); no longer J7.4, L3.2 (K)
- net I2C2_DTA: now also J7.2 (Pin_2); no longer J7.3
- net J3_BOOT0: now also J3.1 (Pin_1)
- net JA: now also JA1.1 (Pin_1)
- net JB: now also JB1.1 (Pin_1)
- net JC: now also JC1.1 (Pin_1)
- net JKA1-1: now also JKA1.1 (Pin_1); no longer J7.2
- net JKA1-2: now also JKA1.2 (Pin_2); no longer J7.1
- net MTRON: now also MO1.3 (Pin_3), J5.1 (Pin_1); no longer MO1.5
- net NRST: now also J4.2 (Pin_2)
- net SEL: now also L4.1 (K), MO1.2 (Pin_2); no longer L4.2 (K), MO1.6
- net SWCLK: now also J10.3 (Pin_3)
- net SWDIO: now also J10.4 (Pin_4)
- net U3-40-PC9: now also JK1.2 (Pin_2)
- net USART1_RX: now also J4.1 (Pin_1)
- net USART1_TX: now also J3.3 (Pin_3)
- net at R20.2: now also L4.2 (A); no longer L4.1 (A)
- net at L5.2 (A), R21.2: now also L3.2 (A); no longer L3.1 (A)
- net D+: no longer names the net of P3.3 (D+), R1.2
- net D-: no longer names the net of P3.2 (D-), R2.2
- no-connect marks 17 -> 16
Other:
- note removed: "JD"
- note removed: "JE"
- title: Gotek(?) SMD Handrawn Schematic, Layout and Gerbers -> Gotek(?) Handrawn Schematic, Layout and Gerbers
- moved on the sheet: C1, C16, C3, C4, C5, C6, C8, C9, R1, R10, R13, R2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
